File: audio_in.kicad_sch (KiCad schematic)
At the start: 17 parts, among them SW1 SW_SPDT

Commit message: Changed D2 and D3 to smaller 0603 diode, changed and rerouted for 4 layers
Parts:
- D2, D3: value SMBJ5.0A-TP -> CG0603MLC-05E; footprint Diode_SMD:D_SMB_Handsoldering -> Diode_SMD:D_0603_1608Metric_Pad1.05x0.95mm_HandSolder
Changed lines of the file:
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@@
       (effects (font (size 1.27 1.27)) (justify right))
     )
-    (property "Value" "SMBJ5.0A-TP" (at 125.73 88.265 90)
+    (property "Value" "CG0603MLC-05E" (at 125.73 88.265 90)
       (effects (font (size 1.27 1.27)) (justify right))
     )
-    (property "Footprint" "Diode_SMD:D_SMB_Handsoldering" (at 132.08 81.28 0)
+    (property "Footprint" "Diode_SMD:D_0603_1608Metric_Pad1.05x0.95mm_HandSolder" (at 132.08 81.28 0)
       (effects (font (size 1.27 1.27)) hide)
     )
@@
       (effects (font (size 1.27 1.27)) (justify right))
     )
-    (property "Value" "SMBJ5.0A-TP" (at 125.73 90.17 90)
+    (property "Value" "CG0603MLC-05E" (at 125.73 90.17 90)
       (effects (font (size 1.27 1.27)) (justify right))
     )
-    (property "Footprint" "Diode_SMD:D_SMB_Handsoldering" (at 128.905 81.28 0)
+    (property "Footprint" "Diode_SMD:D_0603_1608Metric_Pad1.05x0.95mm_HandSolder" (at 128.905 81.28 0)
       (effects (font (size 1.27 1.27)) hide)
     )
