File: stereo_mic_pre.kicad_sch (KiCad schematic)
At the start: 3 parts, among them J1 AudioJack3, J2 AudioJack3

Commit message: Changed D2 and D3 to smaller 0603 diode, changed and rerouted for 4 layers
Connections:
- net audio_in/IN_GND renamed GND_SIG
Other:
- moved on the sheet: J1
Changed lines of the file:
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@@
 (kicad_sch (version 20230121) (generator eeschema)
   (paper "A4")
+  (junction (at 91.44 62.23) (diameter 0) (color 0 0 0 0)
+  )
   (junction (at 91.44 69.85) (diameter 0) (color 0 0 0 0)
   )
+  (junction (at 95.25 69.85) (diameter 0) (color 0 0 0 0)
+  )
+  (junction (at 44.45 114.3) (diameter 0) (color 0 0 0 0)
+  )
   (wire (pts (xy 128.27 61.595) (xy 139.7 61.595))
     (stroke (width 0) (type default))
@@
     (stroke (width 0) (type default))
   )
+  (wire (pts (xy 95.25 69.85) (xy 107.95 69.85))
+    (stroke (width 0) (type default))
+  )
   (wire (pts (xy 91.44 69.85) (xy 91.44 91.44))
     (stroke (width 0) (type default))
@@
     (stroke (width 0) (type default))
   )
+  (wire (pts (xy 95.25 59.055) (xy 95.25 69.85))
+    (stroke (width 0) (type default))
+  )
   (wire (pts (xy 87.63 87.63) (xy 87.63 73.66))
     (stroke (width 0) (type default))
@@
     (stroke (width 0) (type default))
   )
+  (wire (pts (xy 91.44 62.23) (xy 107.95 62.23))
+    (stroke (width 0) (type default))
+  )
   (wire (pts (xy 130.81 65.405) (xy 130.81 64.135))
     (stroke (width 0) (type default))
@@
     (stroke (width 0) (type default))
   )
-  (wire (pts (xy 53.34 111.76) (xy 43.18 111.76))
+  (wire (pts (xy 44.45 114.3) (xy 40.64 114.3))
+    (stroke (width 0) (type default))
+  )
+  (wire (pts (xy 53.34 111.76) (xy 40.64 111.76))
     (stroke (width 0) (type default))
   )
@@
     (stroke (width 0) (type default))
   )
+  (wire (pts (xy 80.01 62.23) (xy 91.44 62.23))
+    (stroke (width 0) (type default))
+  )
   (wire (pts (xy 80.01 73.66) (xy 87.63 73.66))
     (stroke (width 0) (type default))
@@
     (stroke (width 0) (type default))
   )
+  (wire (pts (xy 44.45 114.3) (xy 44.45 119.38))
+    (stroke (width 0) (type default))
+  )
   (wire (pts (xy 38.1 69.85) (xy 57.15 69.85))
     (stroke (width 0) (type default))
@@
     (stroke (width 0) (type default))
   )
-  (wire (pts (xy 43.18 109.22) (xy 57.15 109.22))
+  (wire (pts (xy 40.64 109.22) (xy 57.15 109.22))
     (stroke (width 0) (type default))
   )
@@
     (stroke (width 0) (type default))
   )
-  (wire (pts (xy 91.44 69.85) (xy 107.95 69.85))
-    (stroke (width 0) (type default))
-  )
-  (wire (pts (xy 80.01 62.23) (xy 107.95 62.23))
-    (stroke (width 0) (type default))
-  )
-  (wire (pts (xy 49.53 114.3) (xy 43.18 114.3))
+  (wire (pts (xy 91.44 69.85) (xy 95.25 69.85))
+    (stroke (width 0) (type default))
+  )
+  (wire (pts (xy 91.44 58.42) (xy 91.44 62.23))
+    (stroke (width 0) (type default))
+  )
+  (wire (pts (xy 49.53 114.3) (xy 44.45 114.3))
     (stroke (width 0) (type default))
   )
@@
   (wire (pts (xy 38.1 62.23) (xy 57.15 62.23))
     (stroke (width 0) (type default))
+  )
+  (global_label "GND_VIRT" (shape input) (at 95.25 59.055 90) (fields_autoplaced)
+    (effects (font (size 1.27 1.27)) (justify left))
+    (property "Intersheetrefs" "${INTERSHEET_REFS}" (at 95.25 47.3801 90)
+      (effects (font (size 1.27 1.27)) (justify left) hide)
+    )
+  )
+  (global_label "GND_SIG" (shape input) (at 44.45 119.38 270) (fields_autoplaced)
+    (effects (font (size 1.27 1.27)) (justify right))
+    (property "Intersheetrefs" "${INTERSHEET_REFS}" (at 44.45 130.2082 90)
+      (effects (font (size 1.27 1.27)) (justify right) hide)
+    )
+  )
+  (global_label "VDD_VIRT" (shape input) (at 91.44 58.42 90) (fields_autoplaced)
+    (effects (font (size 1.27 1.27)) (justify left))
+    (property "Intersheetrefs" "${INTERSHEET_REFS}" (at 91.44 46.987 90)
+      (effects (font (size 1.27 1.27)) (justify left) hide)
+    )
   )
   (symbol (lib_id "Device:Battery_Cell") (at 38.1 67.31 0) (unit 1)
@@
     )
   )
-  (symbol (lib_id "Connector:AudioJack3") (at 38.1 111.76 0) (mirror x) (unit 1)
+  (symbol (lib_id "Connector:AudioJack3") (at 35.56 111.76 0) (mirror x) (unit 1)
     (in_bom yes) (on_board yes) (dnp no)
-    (property "Reference" "J1" (at 38.1 120.65 0)
-      (effects (font (size 1.27 1.27)))
-    )
-    (property "Value" "AudioJack3" (at 38.1 118.11 0)
-      (effects (font (size 1.27 1.27)))
-    )
-    (property "Footprint" "Connector_Audio:Jack_3.5mm_CUI_SJ1-3533NG_Horizontal" (at 38.1 111.76 0)
-      (effects (font (size 1.27 1.27)) hide)
-    )
-    (property "Datasheet" "~" (at 38.1 111.76 0)
-      (effects (font (size 1.27 1.27)) hide)
-    )
+    (property "Reference" "J1" (at 35.56 120.65 0)
+      (effects (font (size 1.27 1.27)))
+    )
+    (property "Value" "AudioJack3" (at 35.56 118.11 0)
+      (effects (font (size 1.27 1.27)))
+    )
+    (property "Footprint" "Connector_Audio:Jack_3.5mm_CUI_SJ1-3533NG_Horizontal" (at 35.56 111.76 0)
+      (effects (font (size 1.27 1.27)) hide)
+    )
+    (property "Datasheet" "~" (at 35.56 111.76 0)
+      (effects (font (size 1.27 1.27)) hide)
+    )
